File: Hardware/Top/Tau-TOP.brd (EAGLE design)
At the start: 38 x 38 mm, 52 parts, among them SW1 SWITCH.MOM, SW2 SWITCH.MOM, SW5 SWITCH.MOM, U3 PCF8523, U4 NRF52832_MODULE_MDBT42

Commit message: Changes committed to top and bottom boards
Parts:
- removed SW1, SW2, SW5: SWITCH.MOM, LinnesLab-Switches:TACTILE_SWITCH_SMD_6.2MM_TALL
- added U$1, U$2: SWITCH.MOM, LinnesLab-Switches:TACTILE_SWITCH_SMD_6.2MM_TALL
- moved C2 27.6 mm to (8.13, 29.0)
- moved U3 27.6 mm to (6.27, 25.0)
- moved R6 27.6 mm to (13.7, 24.3)
- moved R5 27.6 mm to (11.4, 25.6)
- moved XTAL3 25.9 mm to (1.75, 23.5)
- moved D5 7.99 mm to (9.75, 9.47)
- moved C5 6.38 mm to (7.24, 2.34)
- moved LDO2 6.06 mm to (10.6, 2.95)
- moved C21 5.96 mm to (20.0, 17.3)
- moved C6 5.88 mm to (13.9, 3.28)
- moved R15 5.84 mm to (16.0, 2.77)
- moved D4 4.27 mm to (9.73, 7.80)
- moved R3 4.12 mm to (2.51, 20.7)
- moved R4 3.18 mm to (5.54, 17.1)
- moved R13 3.17 mm to (6.73, 11.6)
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Connections:
- net VBATT renamed VBAT
- removed net N$11: SW1.A1
- removed net N$9: SW1.B1, SW1.B2
- new net SW1: U$1.A1, U$2.A1
- net GND: now also U$1.B1, U$1.B2, U$2.B1, U$2.B2, USB2.S1, USB2.S2, USB2.S3, USB2.S4, USB2.S5, USB2.S6
