File: Hardware/Top/Tau-TOP.sch (EAGLE design)
At the start: 52 parts, among them SW1 SWITCH.MOM, SW2 SWITCH.MOM, SW5 SWITCH.MOM, U3 PCF8523, U4 NRF52832_MODULE_MDBT42

Commit message: Changes committed to top and bottom boards
Parts:
- removed SW2, SW5: SWITCH.MOM, LinnesLab-Switches:SWITCH.MOM
- added U$2: SWITCH.MOM, LinnesLab-Switches:SWITCH.MOM
- renumbered SW1 to U$1
Connections:
- removed net N$11: U$1.1
- removed net N$9: U$1.3, U$1.4
- removed net VBATT: U3.VBAT
- new net SW1: U$1.1, U$2.1
- net GND: now also U$1.3, U$1.4, U$2.3, U$2.4, USB2.SHIELD
Other:
- note added: "Digital GPIO (general purpose input output) Digital Outputs CS.OLED RESET.OLED DC.OLED [SPI] [I2C] SD.CS Card detect (optional) Digital inputs 3x buttons charge status Analog Inputs Battery monitor Analog Ouputs"
- note added: "Real-Time Clock"
- note added: "nRF52832 Module"
- note removed: "Real-Time Check"
- note removed: "mRFS2832 Module"
Changed lines of the file:
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@@
 <attribute name="MFN_MANUFACTURER" value="NXP USA Inc."/>
 </part>
-<part name="SW1" library="LinnesLab-Switches" deviceset="SWITCH.MOM" device=""/>
-<part name="SW2" library="LinnesLab-Switches" deviceset="SWITCH.MOM" device=""/>
-<part name="SW5" library="LinnesLab-Switches" deviceset="SWITCH.MOM" device=""/>
+<part name="U$1" library="LinnesLab-Switches" deviceset="SWITCH.MOM" device=""/>
+<part name="GND1" library="LinnesLab-Symbols" deviceset="GND" device=""/>
+<part name="U$2" library="LinnesLab-Switches" deviceset="SWITCH.MOM" device=""/>
+<part name="GND3" library="LinnesLab-Symbols" deviceset="GND" device=""/>
 </parts>
 <sheets>
@@
 battery
 if desired</text>
-<text x="-33.02" y="76.2" size="5.08" layer="91">mRFS2832 Module</text>
+<text x="-33.02" y="76.2" size="5.08" layer="91">nRF52832 Module</text>
 <text x="12.7" y="-200.66" size="5.08" layer="91">SD card</text>
 <text x="137.16" y="81.28" size="5.08" layer="91">Cortex Debugger/Programmer</text>
 <text x="182.88" y="25.4" size="5.08" layer="91">RTC</text>
 <text x="162.56" y="-71.12" size="5.08" layer="91">Power Management</text>
-<text x="208.28" y="-269.24" size="5.08" layer="91">Switches</text>
-<text x="149.86" y="-195.58" size="5.08" layer="91">Real-Time Check</text>
+<text x="160.02" y="-261.62" size="5.08" layer="91">Switches</text>
+<text x="119.38" y="-210.82" size="5.08" layer="91">Real-Time Clock</text>
+<text x="-269.24" y="-63.5" size="5.08" layer="94">Digital GPIO (general purpose input output)
+Digital Outputs
+CS.OLED
+RESET.OLED
+DC.OLED
+[SPI]
+[I2C]
+SD.CS
+Card detect (optional)
+Digital inputs
+3x buttons
+charge status
+Analog Inputs
+Battery monitor
+Analog Ouputs</text>
+<wire x1="-116.84" y1="111.76" x2="276.86" y2="111.76" width="0.1524" layer="94"/>
+<wire x1="276.86" y1="111.76" x2="276.86" y2="-320.04" width="0.1524" layer="94"/>
+<wire x1="276.86" y1="-320.04" x2="-116.84" y2="-320.04" width="0.1524" layer="94"/>
+<wire x1="-116.84" y1="-320.04" x2="-116.84" y2="111.76" width="0.254" layer="94"/>
+<wire x1="-109.22" y1="99.06" x2="264.16" y2="99.06" width="0.1524" layer="94" style="longdash"/>
+<wire x1="264.16" y1="99.06" x2="264.16" y2="-35.56" width="0.1524" layer="94" style="longdash"/>
+<wire x1="264.16" y1="-35.56" x2="264.16" y2="-180.34" width="0.1524" layer="94" style="longdash"/>
+<wire x1="264.16" y1="-180.34" x2="264.16" y2="-309.88" width="0.1524" layer="94" style="longdash"/>
+<wire x1="264.16" y1="-309.88" x2="73.66" y2="-309.88" width="0.1524" layer="94" style="longdash"/>
+<wire x1="73.66" y1="-309.88" x2="-109.22" y2="-309.88" width="0.1524" layer="94" style="longdash"/>
+<wire x1="-109.22" y1="-309.88" x2="-109.22" y2="-180.34" width="0.1524" layer="94" style="longdash"/>
+<wire x1="-109.22" y1="-180.34" x2="-109.22" y2="-68.58" width="0.1524" layer="94" style="longdash"/>
+<wire x1="-109.22" y1="-68.58" x2="-109.22" y2="99.06" width="0.1524" layer="94" style="longdash"/>
+<wire x1="127" y1="96.52" x2="127" y2="-35.56" width="0.1524" layer="94" style="longdash"/>
+<wire x1="127" y1="-35.56" x2="264.16" y2="-35.56" width="0.1524" layer="94" style="longdash"/>
+<wire x1="127" y1="-35.56" x2="127" y2="-68.58" width="0.1524" layer="94" style="longdash"/>
+<wire x1="127" y1="-68.58" x2="-109.22" y2="-68.58" width="0.1524" layer="94" style="longdash"/>
+<wire x1="73.66" y1="-71.12" x2="73.66" y2="-180.34" width="0.1524" layer="94" style="longdash"/>
+<wire x1="73.66" y1="-180.34" x2="264.16" y2="-180.34" width="0.1524" layer="94" style="longdash"/>
+<wire x1="73.66" y1="-180.34" x2="-109.22" y2="-180.34" width="0.1524" layer="94" style="longdash"/>
+<wire x1="73.66" y1="-180.34" x2="73.66" y2="-309.88" width="0.1524" layer="94" style="longdash"/>
 </plain>
 <instances>
@@
 <attribute name="MFN_MANUFACTURER" x="144.78" y="-233.68" size="1.27" layer="96" display="off"/>
 </instance>
-<instance part="SW1" gate="G$1" x="127" y="-274.32" smashed="yes">
+<instance part="U$1" gate="G$1" x="127" y="-274.32" smashed="yes">
 <attribute name="NAME" x="127" y="-269.494" size="1.778" layer="95" font="vector" align="bottom-center"/>
 <attribute name="VALUE" x="127" y="-277.114" size="1.778" layer="96" font="vector" align="top-center"/>
 </instance>
-<instance part="SW2" gate="G$1" x="149.86" y="-276.86" smashed="yes">
-<attribute name="NAME" x="149.86" y="-272.034" size="1.778" layer="95" font="vector" align="bottom-center"/>
-<attribute name="VALUE" x="149.86" y="-279.654" size="1.778" layer="96" font="vector" align="top-center"/>
-</instance>
-<instance part="SW5" gate="G$1" x="190.5" y="-279.4" smashed="yes">
-<attribute name="NAME" x="190.5" y="-274.574" size="1.778" layer="95" font="vector" align="bottom-center"/>
-<attribute name="VALUE" x="190.5" y="-282.194" size="1.778" layer="96" font="vector" align="top-center"/>
+<instance part="GND1" gate="G$1" x="134.62" y="-281.94" smashed="yes">
+<attribute name="VALUE" x="134.62" y="-282.194" size="1.778" layer="96" align="top-center"/>
+</instance>
+<instance part="U$2" gate="G$1" x="154.94" y="-274.32" smashed="yes">
+<attribute name="NAME" x="154.94" y="-269.494" size="1.778" layer="95" font="vector" align="bottom-center"/>
+<attribute name="VALUE" x="154.94" y="-277.114" size="1.778" layer="96" font="vector" align="top-center"/>
+</instance>
+<instance part="GND3" gate="G$1" x="162.56" y="-281.94" smashed="yes">
+<attribute name="VALUE" x="162.56" y="-282.194" size="1.778" layer="96" align="top-center"/>
 </instance>
 </instances>
@@
 <pinref part="GND25" gate="G$1" pin="GND"/>
 <wire x1="137.16" y1="-137.16" x2="137.16" y2="-144.78" width="0.1524" layer="91"/>
+<pinref part="USB2" gate="G$1" pin="SHIELD"/>
+<wire x1="134.62" y1="-124.46" x2="137.16" y2="-124.46" width="0.1524" layer="91"/>
+<wire x1="137.16" y1="-124.46" x2="137.16" y2="-137.16" width="0.1524" layer="91"/>
+<junction x="137.16" y="-137.16"/>
 </segment>
 <segment>
@@
 <pinref part="GND5" gate="G$1" pin="GND"/>
 <pinref part="C2" gate="G$1" pin="2"/>
+</segment>
+<segment>
+<pinref part="U$1" gate="G$1" pin="3"/>
+<wire x1="132.08" y1="-274.32" x2="134.62" y2="-274.32" width="0.1524" layer="91"/>
+<wire x1="134.62" y1="-279.4" x2="134.62" y2="-276.86" width="0.1524" layer="91"/>
+<pinref part="U$1" gate="G$1" pin="4"/>
+<wire x1="134.62" y1="-276.86" x2="134.62" y2="-274.32" width="0.1524" layer="91"/>
+<wire x1="132.08" y1="-276.86" x2="134.62" y2="-276.86" width="0.1524" layer="91"/>
+<junction x="134.62" y="-276.86"/>
+<pinref part="GND1" gate="G$1" pin="GND"/>
+</segment>
+<segment>
+<pinref part="U$2" gate="G$1" pin="3"/>
+<wire x1="160.02" y1="-274.32" x2="162.56" y2="-274.32" width="0.1524" layer="91"/>
+<wire x1="162.56" y1="-279.4" x2="162.56" y2="-276.86" width="0.1524" layer="91"/>
+<pinref part="U$2" gate="G$1" pin="4"/>
+<wire x1="162.56" y1="-276.86" x2="162.56" y2="-274.32" width="0.1524" layer="91"/>
+<wire x1="160.02" y1="-276.86" x2="162.56" y2="-276.86" width="0.1524" layer="91"/>
+<junction x="162.56" y="-276.86"/>
+<pinref part="GND3" gate="G$1" pin="GND"/>
 </segment>
 </net>
@@
 </segment>
 </net>
-<net name="VBATT" class="0">
-<segment>
-<wire x1="129.54" y1="-236.22" x2="127" y2="-236.22" width="0.1524" layer="91"/>
-<label x="127" y="-236.22" size="1.27" layer="95" rot="R180" xref="yes"/>
-<pinref part="U3" gate="G$1" pin="VBAT"/>
-</segment>
-</net>
-<net name="N$9" class="0">
-<segment>
-<pinref part="SW1" gate="G$1" pin="3"/>
-<wire x1="132.08" y1="-274.32" x2="134.62" y2="-274.32" width="0.1524" layer="91"/>
-<wire x1="134.62" y1="-274.32" x2="134.62" y2="-276.86" width="0.1524" layer="91"/>
-<pinref part="SW1" gate="G$1" pin="4"/>
-<wire x1="134.62" y1="-284.48" x2="134.62" y2="-276.86" width="0.1524" layer="91"/>
-<wire x1="134.62" y1="-276.86" x2="132.08" y2="-276.86" width="0.1524" layer="91"/>
-</segment>
-</net>
-<net name="N$11" class="0">
-<segment>
-<pinref part="SW1" gate="G$1" pin="1"/>
+<net name="SW1" class="0">
+<segment>
+<pinref part="U$1" gate="G$1" pin="1"/>
 <wire x1="121.92" y1="-274.32" x2="119.38" y2="-274.32" width="0.1524" layer="91"/>
-</segment>
-</net>
+<label x="119.38" y="-274.32" size="1.27" layer="95" ratio="15" rot="R180" xref="yes"/>
+</segment>
+<segment>
+<pinref part="U$2" gate="G$1" pin="1"/>
+<wire x1="149.86" y1="-274.32" x2="147.32" y2="-274.32" width="0.1524" layer="91"/>
+<label x="147.32" y="-274.32" size="1.27" layer="95" ratio="15" rot="R180" xref="yes"/>
+</segment>
+</net>

Commit message: Changes committed to the top and bottom board. Connections between the two have been noted as well
Parts:
- added C15: 100n, LinnesLab-Passives:CAPACITOR0603
- added C16, C17: 47p, LinnesLab-Passives:CAPACITOR0603
- added JP2: (no value), LinnesLab-Switches:JUMPER-SMT_2_NO_SILK
- added LED5: RED, LinnesLab-LED:LED0603
- added LED6: YELLOW, LinnesLab-LED:LED0603
- added R1, R2: 0, LinnesLab-Passives:RESISTOR0603
- added R17, R18: 27, LinnesLab-Passives:RESISTOR0603
- added R19, R20: 1k, LinnesLab-Passives:RESISTOR0603
- added U5: FT231XS, LinnesLab-DigitalIC:FT231XS
Connections:
- removed net RXD: U4.P0.08
- removed net TXD: U4.P0.06
- new net !CTS: JP2.2, U5.!CTS
- new net FT3V3: U5.3V3OUT
- new net N$22: R17.2, U5.USBDM
- new net N$24: R18.2, U5.USBDP
- new net N$25: LED5.C, R19.2
- new net N$26: LED6.C, R20.2
- new net RXD.FT: R2.1, U5.RXD
- new net RXD.NRF: R1.2, U4.P0.08
- new net RXLED: R19.1, U5.CBUS1
- new net TXD.FT: R1.1, U5.TXD
- new net TXD.NRF: R2.2, U4.P0.06
- new net TXLED: R20.1, U5.CBUS2
- net 3.3V: now also C15.2, LED5.A, LED6.A, U5.!RESET, U5.VCCIO
- net DTR: now also U5.!DTR
- net GND: now also C15.1, C16.2, C17.1, JP2.1, U5.GND@16, U5.GND@6
- net SCL: now also R6.1; no longer R5.1
- net SDA: now also R5.1; no longer R6.1
- net USB+: now also C16.1, R18.1
- net USB-: now also C17.2, R17.1
- net V_USB: now also U5.VCC
Other:
- note added: "FTDI-Serial-to-USB converter"
- note added: "I don't remember if CTS needs to be grounded or left floating so here's a jumper to ground so it can be configued either way dynamically."
- note added: "Last text is arduino pin number (digital or analog)"
- note added: "Notes"
- note added: "TXD goes to RX on the other device RXD goes to TX on the other device"
- moved on the sheet: C2, R5, R6, U3, XTAL3

Commit message: Changes committed to top and bottom board
Parts:
- added J1: (no value), LinnesLab-Connectors:CONN_07
Connections:
- removed net BATT: R13.1, R14.2
- removed net CD1: SD2.CARD_DETECT
- removed net CHRG.STAT: CHRG2.STAT, R12.1
- removed net CS.OLED: U2./CS
- removed net DC.OLED: U2.DC/I2C_SA0
- removed net RESET.OLED: U2./RES
- removed net SD.CS: SD2.CS
- removed net SW1: U$1.1, U$2.1
- new net A4/BATT: R13.1, R14.2, U4.P0.28/AIN4
- new net A6/TIA: U4.P0.30/AIN6
- new net A7/PPG: U4.P0.31/AIN7
- new net D11/SW1: U$1.1, U4.P0.11
- new net D15/SW2: U$2.1, U4.P0.15
- new net D16/CS.OLED: U2./CS, U4.P0.16
- new net D27/CHRG.STATUS: CHRG2.STAT, R12.1, U4.P0.27
- new net D29/LED.CTRL: U4.P0.29/AIN5
- new net D3/RESET.OLED: U2./RES, U4.P0.03/AIN1
- new net D4/DC.OLED: U2.DC/I2C_SA0, U4.P0.04/AIN2
- new net D5/CD1: SD2.CARD_DETECT, U4.P0.05/AIN3
- new net D7/SD.CS: SD2.CS, U4.P0.07
Other:
- note added: "Digital Output"
Changed lines of the file:
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@@
 <part name="SUPPLY1" library="LinnesLab-Symbols" deviceset="3.3V" device=""/>
 <part name="SUPPLY4" library="LinnesLab-Symbols" deviceset="3.3V" device=""/>
+<part name="J1" library="LinnesLab-Connectors" deviceset="CONN_07" device=""/>
 </parts>
 <sheets>
@@
 <text x="160.02" y="-261.62" size="5.08" layer="91">Switches</text>
 <text x="119.38" y="-210.82" size="5.08" layer="91">Real-Time Clock</text>
-<text x="-269.24" y="-63.5" size="5.08" layer="94">Digital GPIO (general purpose input output)
+<text x="-185.42" y="127" size="5.08" layer="94">Digital GPIO (general purpose input output)
 Digital Outputs
 CS.OLED
@@
 if desired</text>
 <text x="165.1" y="198.12" size="5.08" layer="91">FTDI-Serial-to-USB converter</text>
-<text x="-271.78" y="73.66" size="10.16" layer="94">Notes</text>
+<text x="-187.96" y="264.16" size="10.16" layer="94">Notes</text>
+<text x="180.34" y="-149.86" size="1.27" layer="95">Digital Output</text>
 </plain>
 <instances>
@@
 <instance part="SUPPLY4" gate="G$1" x="-73.66" y="96.52" smashed="yes">
 <attribute name="VALUE" x="-73.66" y="99.314" size="1.778" layer="96" align="bottom-center"/>
+</instance>
+<instance part="J1" gate="G$1" x="-45.72" y="99.06" smashed="yes">
+<attribute name="VALUE" x="-50.8" y="89.154" size="1.778" layer="96" font="vector"/>
+<attribute name="NAME" x="-50.8" y="112.268" size="1.778" layer="95" font="vector"/>
 </instance>
 </instances>
@@
 </segment>
 </net>
-<net name="DC.OLED" class="0">
-<segment>
-<label x="-20.32" y="-132.08" size="1.778" layer="95"/>
-<pinref part="U2" gate="G$1" pin="DC/I2C_SA0"/>
-<wire x1="5.08" y1="-132.08" x2="-20.32" y2="-132.08" width="0.1524" layer="91"/>
-</segment>
-</net>
-<net name="RESET.OLED" class="0">
-<segment>
-<label x="-20.32" y="-129.54" size="1.778" layer="95"/>
-<pinref part="U2" gate="G$1" pin="/RES"/>
-<wire x1="5.08" y1="-129.54" x2="-20.32" y2="-129.54" width="0.1524" layer="91"/>
-</segment>
-</net>
 <net name="N$1" class="0">
 <segment>
@@
 </segment>
 </net>
-<net name="CS.OLED" class="0">
-<segment>
-<label x="-20.32" y="-127" size="1.778" layer="95"/>
-<pinref part="U2" gate="G$1" pin="/CS"/>
-<wire x1="5.08" y1="-127" x2="-20.32" y2="-127" width="0.1524" layer="91"/>
-</segment>
-</net>
 <net name="CD2" class="0">
 <segment>
@@
 <label x="-5.08" y="-220.98" size="1.27" layer="95" rot="R180" xref="yes"/>
 <pinref part="SD2" gate="G$1" pin="CARD_DETECT1"/>
-</segment>
-</net>
-<net name="CD1" class="0">
-<segment>
-<wire x1="-5.08" y1="-218.44" x2="0" y2="-218.44" width="0.1524" layer="91"/>
-<label x="-5.08" y="-218.44" size="1.27" layer="95" rot="R180" xref="yes"/>
-<pinref part="SD2" gate="G$1" pin="CARD_DETECT"/>
-</segment>
-</net>
-<net name="SD.CS" class="0">
-<segment>
-<wire x1="-5.08" y1="-236.22" x2="0" y2="-236.22" width="0.1524" layer="91"/>
-<label x="-5.08" y="-236.22" size="1.27" layer="95" rot="R180" xref="yes"/>
-<pinref part="SD2" gate="G$1" pin="CS"/>
 </segment>
 </net>
@@
 </segment>
 </net>
-<net name="CHRG.STAT" class="0">
-<segment>
-<pinref part="R12" gate="G$1" pin="1"/>
-<wire x1="175.26" y1="-139.7" x2="175.26" y2="-144.78" width="0.1524" layer="91"/>
-<wire x1="175.26" y1="-144.78" x2="180.34" y2="-144.78" width="0.1524" layer="91"/>
-<wire x1="180.34" y1="-144.78" x2="180.34" y2="-132.08" width="0.1524" layer="91"/>
-<pinref part="CHRG2" gate="G$1" pin="STAT"/>
-<wire x1="180.34" y1="-132.08" x2="182.88" y2="-132.08" width="0.1524" layer="91"/>
-<label x="180.34" y="-144.78" size="1.27" layer="95" xref="yes"/>
-</segment>
-</net>
 <net name="USB-" class="0">
 <segment>
@@
 <junction x="157.48" y="149.86"/>
 <label x="144.78" y="149.86" size="1.27" layer="95" rot="R180" xref="yes"/>
-</segment>
-</net>
-<net name="BATT" class="0">
-<segment>
-<pinref part="R13" gate="G$1" pin="1"/>
-<pinref part="R14" gate="G$1" pin="2"/>
-<wire x1="236.22" y1="-116.84" x2="236.22" y2="-109.22" width="0.1524" layer="91"/>
-<label x="236.22" y="-114.3" size="1.27" layer="95" xref="yes"/>
 </segment>
 </net>
@@
 </segment>
 </net>
-<net name="SW1" class="0">
-<segment>
-<pinref part="U$1" gate="G$1" pin="1"/>
-<wire x1="121.92" y1="-274.32" x2="119.38" y2="-274.32" width="0.1524" layer="91"/>
-<label x="119.38" y="-274.32" size="1.27" layer="95" ratio="15" rot="R180" xref="yes"/>
-</segment>
+<net name="D15/SW2" class="0">
 <segment>
 <pinref part="U$2" gate="G$1" pin="1"/>
 <wire x1="149.86" y1="-274.32" x2="147.32" y2="-274.32" width="0.1524" layer="91"/>
 <label x="147.32" y="-274.32" size="1.27" layer="95" ratio="15" rot="R180" xref="yes"/>
+</segment>
+<segment>
+<pinref part="U4" gate="G$1" pin="P0.15"/>
+<wire x1="17.78" y1="20.32" x2="20.32" y2="20.32" width="0.1524" layer="91"/>
+<label x="20.32" y="20.32" size="1.27" layer="95" xref="yes"/>
 </segment>
 </net>
@@
 </segment>
 </net>
+<net name="D27/CHRG.STATUS" class="0">
+<segment>
+<pinref part="U4" gate="G$1" pin="P0.27"/>
+<wire x1="-27.94" y1="30.48" x2="-30.48" y2="30.48" width="0.1524" layer="91" style="longdash"/>
+<label x="-30.48" y="30.48" size="1.27" layer="95" rot="R180" xref="yes"/>
+</segment>
+<segment>
+<pinref part="R12" gate="G$1" pin="1"/>
+<wire x1="175.26" y1="-139.7" x2="175.26" y2="-144.78" width="0.1524" layer="91"/>
+<wire x1="175.26" y1="-144.78" x2="180.34" y2="-144.78" width="0.1524" layer="91"/>
+<wire x1="180.34" y1="-144.78" x2="180.34" y2="-132.08" width="0.1524" layer="91"/>
+<pinref part="CHRG2" gate="G$1" pin="STAT"/>
+<wire x1="180.34" y1="-132.08" x2="182.88" y2="-132.08" width="0.1524" layer="91"/>
+<label x="180.34" y="-144.78" size="1.27" layer="95" xref="yes"/>
+</segment>
+</net>
+<net name="A4/BATT" class="0">
+<segment>
+<pinref part="U4" gate="G$1" pin="P0.28/AIN4"/>
+<wire x1="-27.94" y1="27.94" x2="-30.48" y2="27.94" width="0.1524" layer="91" style="longdash"/>
+<label x="-30.48" y="27.94" size="1.27" layer="95" rot="R180" xref="yes"/>
+</segment>
+<segment>
+<pinref part="R13" gate="G$1" pin="1"/>
+<pinref part="R14" gate="G$1" pin="2"/>
+<wire x1="236.22" y1="-116.84" x2="236.22" y2="-109.22" width="0.1524" layer="91"/>
+<label x="236.22" y="-114.3" size="1.27" layer="95" xref="yes"/>
+</segment>
+</net>
+<net name="D7/SD.CS" class="0">
+<segment>
+<pinref part="U4" gate="G$1" pin="P0.07"/>
+<wire x1="0" y1="-2.54" x2="0" y2="-5.08" width="0.1524" layer="91"/>
+<label x="0" y="-5.08" size="1.27" layer="95" rot="R270" xref="yes"/>
+</segment>
+<segment>
+<wire x1="-5.08" y1="-236.22" x2="0" y2="-236.22" width="0.1524" layer="91"/>
+<label x="-5.08" y="-236.22" size="1.27" layer="95" rot="R180" xref="yes"/>
+<pinref part="SD2" gate="G$1" pin="CS"/>
+</segment>
+</net>
+<net name="D5/CD1" class="0">
+<segment>
+<pinref part="U4" gate="G$1" pin="P0.05/AIN3"/>
+<wire x1="-5.08" y1="-2.54" x2="-5.08" y2="-5.08" width="0.1524" layer="91"/>
+<label x="-5.08" y="-5.08" size="1.27" layer="95" rot="R270" xref="yes"/>
+</segment>
+<segment>
+<wire x1="-5.08" y1="-218.44" x2="0" y2="-218.44" width="0.1524" layer="91"/>
+<label x="-5.08" y="-218.44" size="1.27" layer="95" rot="R180" xref="yes"/>
+<pinref part="SD2" gate="G$1" pin="CARD_DETECT"/>
+</segment>
+</net>
+<net name="D11/SW1" class="0">
+<segment>
+<pinref part="U4" gate="G$1" pin="P0.11"/>
+<wire x1="17.78" y1="10.16" x2="20.32" y2="10.16" width="0.1524" layer="91"/>
+<label x="20.32" y="10.16" size="1.27" layer="95" xref="yes"/>
+</segment>
+<segment>
+<pinref part="U$1" gate="G$1" pin="1"/>
+<wire x1="121.92" y1="-274.32" x2="119.38" y2="-274.32" width="0.1524" layer="91"/>
+<label x="119.38" y="-274.32" size="1.27" layer="95" ratio="15" rot="R180" xref="yes"/>
+</segment>
+</net>
+<net name="D16/CS.OLED" class="0">
+<segment>
+<pinref part="U4" gate="G$1" pin="P0.16"/>
+<wire x1="17.78" y1="22.86" x2="20.32" y2="22.86" width="0.1524" layer="91"/>
+<label x="20.32" y="22.86" size="1.27" layer="95" xref="yes"/>
+</segment>
+<segment>
+<label x="-20.32" y="-127" size="1.778" layer="95"/>
+<pinref part="U2" gate="G$1" pin="/CS"/>
+<wire x1="5.08" y1="-127" x2="-20.32" y2="-127" width="0.1524" layer="91"/>
+</segment>
+</net>
+<net name="D3/RESET.OLED" class="0">
+<segment>
+<pinref part="U4" gate="G$1" pin="P0.03/AIN1"/>
+<wire x1="-10.16" y1="-2.54" x2="-10.16" y2="-5.08" width="0.1524" layer="91"/>
+<label x="-10.16" y="-5.08" size="1.27" layer="95" rot="R270" xref="yes"/>
+</segment>
+<segment>
+<label x="-20.32" y="-129.54" size="1.778" layer="95"/>
+<pinref part="U2" gate="G$1" pin="/RES"/>
+<wire x1="5.08" y1="-129.54" x2="-20.32" y2="-129.54" width="0.1524" layer="91"/>
+</segment>
+</net>
+<net name="D4/DC.OLED" class="0">
+<segment>
+<pinref part="U4" gate="G$1" pin="P0.04/AIN2"/>
+<wire x1="-7.62" y1="-2.54" x2="-7.62" y2="-5.08" width="0.1524" layer="91"/>
+<label x="-7.62" y="-5.08" size="1.27" layer="95" rot="R270" xref="yes"/>
+</segment>
+<segment>
+<label x="-20.32" y="-132.08" size="1.778" layer="95"/>
+<pinref part="U2" gate="G$1" pin="DC/I2C_SA0"/>
+<wire x1="5.08" y1="-132.08" x2="-20.32" y2="-132.08" width="0.1524" layer="91"/>
+</segment>
+</net>
+<net name="D29/LED.CTRL" class="0">
+<segment>
+<pinref part="U4" gate="G$1" pin="P0.29/AIN5"/>
+<wire x1="-27.94" y1="25.4" x2="-30.48" y2="25.4" width="0.1524" layer="91"/>
+<label x="-30.48" y="25.4" size="1.27" layer="95" rot="R180" xref="yes"/>
+</segment>
+</net>
+<net name="A6/TIA" class="0">
+<segment>
+<pinref part="U4" gate="G$1" pin="P0.30/AIN6"/>
+<wire x1="-27.94" y1="22.86" x2="-30.48" y2="22.86" width="0.1524" layer="91"/>
+<label x="-30.48" y="22.86" size="1.27" layer="95" rot="R180" xref="yes"/>
+</segment>
+</net>
+<net name="A7/PPG" class="0">
+<segment>
+<pinref part="U4" gate="G$1" pin="P0.31/AIN7"/>
+<wire x1="-27.94" y1="20.32" x2="-30.48" y2="20.32" width="0.1524" layer="91"/>
+<label x="-30.48" y="20.32" size="1.27" layer="95" rot="R180" xref="yes"/>
+</segment>
+</net>
