File: Hardware/Top/Tau-TOP.sch (EAGLE design)
At the start: 65 parts, among them U3 PCF8523, U4 NRF52832_MODULE_MDBT42, U5 FT231XS

Commit message: Changes made to top and bottom board
Parts:
- removed C22: (no value), LinnesLab-Passives:CAPACITOR0603
- removed C23, C24: 300p, LinnesLab-Passives:CAPACITOR0603
- removed C25: 10u, LinnesLab-Passives:CAPACITOR0805
- removed C26: 100n, LinnesLab-Passives:CAPACITOR0603
- removed D4: (no value), LinnesLab-DiscreteSemi:SCHOTTKY-USC
- removed LED5: RED, LinnesLab-LED:LED0603
- removed LED6: YELLOW, LinnesLab-LED:LED0603
- removed R19, R20: 1k, LinnesLab-Passives:RESISTOR0603
- removed U$2: SWITCH.MOM, LinnesLab-Switches:SWITCH.MOM
- removed U5: FT231XS, LinnesLab-DigitalIC:FT231XS
- removed XTAL3: 32.7680kHz, LinnesLab-Clocks:CRYSTALECS-.327-12.5-12-C-TR
- added C1, C18, C19: 1u, LinnesLab-Passives:CAPACITOR0603
- added C3: (no value), LinnesLab-Passives:CAPACITOR0603
- added C4: 10uF, LinnesLab-Passives:CAPACITOR0603
- added D3: (no value), LinnesLab-DiscreteSemi:SCHOTTKY-USC
- added LED1: RED, LinnesLab-LED:LED0603
- added LED2: BLUE, LinnesLab-LED:LED0603
- added R16: 100k, LinnesLab-Passives:RESISTOR0603
- added R7: 27, LinnesLab-Passives:RESISTOR0603
- added SW1: (no value), LinnesLab-Switches:SPST-PTS830GG140-COPY.1-3
- added XTAL1: 32.768kHz, LinnesLab-Clocks:CRYSTALECS-.327-12.5-12-C-TR
- C11, C12: value 2.2uF -> 300p; device LinnesLab-Passives:CAPACITOR0402 -> LinnesLab-Passives:CAPACITOR0603
- C13, C14: value 4.7u -> 47p
- C16: value 47p -> 4.7u
- C17: value 47p -> 100n
- C2: value 1u -> 10u; device LinnesLab-Passives:CAPACITOR0603 -> LinnesLab-Passives:CAPACITOR0805
- C21: value (none) -> 4.7u
- C5, C6: value 1u -> 2.2uF; device LinnesLab-Passives:CAPACITOR0603 -> LinnesLab-Passives:CAPACITOR0402
- C7: value 2.2uF -> (none); device LinnesLab-Passives:CAPACITOR0402 -> LinnesLab-Passives:CAPACITOR0603
- C9: value 10uF -> 2.2uF; device LinnesLab-Passives:CAPACITOR0603 -> LinnesLab-Passives:CAPACITOR0402
- J1: device LinnesLab-Connectors:CONN_07 -> LinnesLab-Connectors:CONN_07-1.27MM
- LED4: value BLUE -> YELLOW
- R1, R2: value 0 -> 10k
- R13: value 100k -> 1k
- R14, R15: value 100k -> 0
- R17: value 27 -> 100k
- R18: value 27 -> 1k
- R5, R6: value 10k -> 1k
- R8: value 1k -> 27
- R9: value 1k -> 100k
- SW3: value (none) -> SWITCH.MOM; device LinnesLab-Switches:SPST-PTS830GG140-COPY.1-3 -> LinnesLab-Switches:SWITCH.MOM
- U4: value NRF52832_MODULE_MDBT42 -> FT231XS; device LinnesLab-Microcontrollers:NRF52832_MODULE_MDBT42 -> LinnesLab-DigitalIC:FT231XS
- XTAL2: value 32.768kHz -> 32.7680kHz; FREQ (none) -> 32.7680KHZ
- renumbered CHRG2 to CHRG1, CORTEX1 to DEBUG1, D5 to D2, JP2 to JP1, L2 to L1, LDO2 to LDO1, SD2 to SD1, U$1 to SW2, USB2 to USB1
Connections:
- removed net FRST: U4.P0.22
- net !CTS: now also U4.!CTS; no longer U5.!CTS
- net 3.3V: now also C17.2, C19.1, C2.2, C20.1, C9.2, D3.C, J1.4, LED3.A, LED4.A, R1.2, R12.2, R2.2, U4.!RESET, U4.VCCIO; no longer C12.2, C15.2, C2.1, C25.2, C6.1, D1.C, LED5.A, LED6.A, R15.2, R5.2, R6.2, U4.VDD, U5.!RESET, U5.VCCIO
- net A4/BATT: now also R16.1, R17.2; no longer R13.1, R14.2, U4.P0.28/AIN4
- net A6/TIA: now also J1.6; no longer U4.P0.30/AIN6
- net A7/PPG: now also J1.7; no longer U4.P0.31/AIN7
- net D11/SW1: no longer U4.P0.11
- net D15/SW2: now also SW3.1; no longer U$2.1, U4.P0.15
- net D16/CS.OLED: no longer U4.P0.16
- net D27/CHRG.STATUS: now also R9.1; no longer R12.1, U4.P0.27
- net D29/LED.CTRL: now also J1.5; no longer U4.P0.29/AIN5
- net D3/RESET.OLED: no longer U4.P0.03/AIN1
- net D4/DC.OLED: no longer U4.P0.04/AIN2
- net D5/CD1: no longer U4.P0.05/AIN3
- net D7/SD.CS: no longer U4.P0.07
- net DFU: now also SW1.B; no longer SW3.B, U4.P0.20
- net DTR: now also C15.1, U4.!DTR; no longer C26.1, U5.!DTR
- net FT3V3: now also U4.3V3OUT; no longer U5.3V3OUT
- net GND: now also C1.2, C11.2, C12.2, C13.1, C14.2, C16.1, C18.1, C19.2, C2.1, C21.2, C3.1, C4.1, C6.1, C7.2, J1.3, LED1.C, LED2.C, R12.1, R17.1, SW1.A, SW3.3, SW3.4, U4.GND@16, U4.GND@6; no longer C11.1, C12.1, C13.2, C14.1, C15.1, C16.2, C2.2, C21.1, C22.2, C23.2, C24.2, C25.1, C5.1, C6.2, LED3.C, LED4.C, R14.1, R15.1, SW3.A, U$2.3, U$2.4, U4.GND@1, U4.GND@2, U4.GND@3, U4.GND@4, U5.GND@16, U5.GND@6
- net LED1: now also R5.2; no longer R8.2, U4.P0.17
- net LED2: now also R6.2; no longer R9.2, U4.P0.19
- net MISO: no longer U4.P0.14
- net MOSI: no longer U4.P0.13
- net N$12: now also XTAL2.1; no longer XTAL3.1
- net N$13: now also XTAL2.2; no longer XTAL3.2
- net N$16: now also C3.2, XTAL1.1; no longer C21.2, U4.P0.00/XL1, XTAL2.1
- net N$17: now also C7.1, XTAL1.2; no longer C22.1, U4.P0.01/XL2, XTAL2.2
- net N$18: now also LED1.A, R5.1; no longer LED3.A, R8.1
- net N$19: now also LED2.A, R6.1; no longer LED4.A, R9.1
- net N$20: no longer U4.DCC
- net N$21: now also C1.1; no longer C20.1, U4.DEC4
- net N$22: now also R7.2, U4.USBDM; no longer R17.2, U5.USBDM
- net N$24: now also R8.2, U4.USBDP; no longer R18.2, U5.USBDP
- net N$25: now also LED3.C, R13.2; no longer LED5.C, R19.2
- net N$26: now also LED4.C, R18.2; no longer LED6.C, R20.2
- net N$3: now also C8.2; no longer C7.2
- net N$4: now also C8.1; no longer C7.1
- net N$5: now also C5.2; no longer C8.2
- net N$6: now also C5.1; no longer C8.1
- net N$7: now also C4.2; no longer C9.2
- net N$8: now also C6.2; no longer C11.2
- net P0.09/NFC1: now also C11.1; no longer C24.1, U4.P0.09
- net P0.10/NFC2: now also C12.1; no longer C23.1, U4.P0.10
- net RESET: now also C15.2, D3.A; no longer C26.2, D1.A, U4.P0.21/RESET
- net RXD.FT: now also R15.1, U4.RXD; no longer R2.1, U5.RXD
- net RXD.NRF: now also R14.2; no longer R1.2, U4.P0.08
- net RXLED: now also R13.1, U4.CBUS1; no longer R19.1, U5.CBUS1
- net SCK: no longer U4.P0.12
- net SCL: now also J1.2, R2.1; no longer R6.1, U4.P0.26
- net SDA: now also J1.1, R1.1; no longer R5.1, U4.P0.25
- net SWCLK: no longer U4.SWDCLK
- net SWDIO: no longer U4.SWDIO
- net SWO: no longer U4.P0.18/SWO
- net TXD.FT: now also R14.1, U4.TXD; no longer R1.1, U5.TXD
- net TXD.NRF: now also R15.2; no longer R2.2, U4.P0.06
- net TXLED: now also R18.1, U4.CBUS2; no longer R20.1, U5.CBUS2
- net USB+: now also C14.1, R8.1; no longer C16.1, R18.1
- net USB-: now also C13.2, R7.1; no longer C17.2, R17.1
- net VIN: now also C16.2, C18.2, D1.C, R9.2; no longer C14.2, C5.2, D4.C, R12.2
- net VLIPO: now also C21.1, D1.A, R16.2; no longer C13.1, D4.A, R13.2
- net V_USB: now also U4.VCC; no longer U5.VCC
Other:
- note added: "Connection to lower board"
- note added: "Connection to upper board"
- moved on the sheet: C11, C12, C13, C14, C15, C16, C17, C2, C20, C21, C5, C6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

Commit message: Changes made to Top board and arduino files
Parts:
- removed C11, C12: 300p, LinnesLab-Passives:CAPACITOR0603
- added U1: NRF52832_MODULE_MDBT42, LinnesLab-Microcontrollers:NRF52832_MODULE_MDBT42
- C10: value 2.2uF -> (none); device LinnesLab-Passives:CAPACITOR0402 -> LinnesLab-Passives:CAPACITOR0603
- C3: value (none) -> 10uF
- C4: value 10uF -> (none)
- C7: value (none) -> 2.2uF; device LinnesLab-Passives:CAPACITOR0603 -> LinnesLab-Passives:CAPACITOR0402
- XTAL2: FREQ 32.7680KHZ -> (none)
Connections:
- removed net N$16: C3.2, XTAL1.1
- removed net N$17: C7.1, XTAL1.2
- removed net N$20: L1.1
- removed net N$21: C1.1, L1.2
- new net FRST: U1.P0.22
- new net N$31: C4.2, U1.P0.00/XL1, XTAL1.1
- new net N$32: C10.1, U1.P0.01/XL2, XTAL1.2
- new net N$35: L1.1, U1.DCC
- new net N$36: C1.1, L1.2, U1.DEC4
- new net RXD: U1.P0.08
- new net TXD: U1.P0.06
- net 3.3V: now also C8.2, U1.VDD; no longer C10.2
- net DFU: now also U1.P0.20
- net GND: now also C10.2, C8.1, U1.GND@1, U1.GND@2, U1.GND@3, U1.GND@4; no longer C10.1, C11.2, C12.2, C7.2, SW2.4, SW3.4
- net LED1: now also U1.P0.17
- net LED2: now also U1.P0.19
- net MISO: now also U1.P0.14
- net MOSI: now also U1.P0.13
- net N$3: now also C7.2; no longer C8.2
- net N$4: now also C7.1; no longer C8.1
- net N$7: now also C3.2; no longer C4.2
- net P0.09/NFC1: now also U1.P0.09; no longer C11.1
- net P0.10/NFC2: now also U1.P0.10; no longer C12.1
- net RESET: now also U1.P0.21/RESET
- net SCK: now also U1.P0.12
- net SCL: now also U1.P0.26
- net SDA: now also U1.P0.25
- net SWCLK: now also U1.SWDCLK
- net SWDIO: now also U1.SWDIO
- net SWO: now also U1.P0.18/SWO
Other:
- note removed: "Last text is arduino pin number (digital or analog)"
- moved on the sheet: C1, C10, C2, C3, C4, C7, C8, C9, L1, LED1, LED2, R5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

Commit message: Changes made to top and bottom board
Parts:
- removed C19: 1u, LinnesLab-Passives:CAPACITOR0603
- removed C21: 4.7u, LinnesLab-Passives:CAPACITOR0603
- removed SD1: (no value), LinnesLab-Connectors:MICROSD
- removed U3: PCF8523, LinnesLab-Clocks:PCF8523
- removed XTAL2: 32.7680kHz, LinnesLab-Clocks:CRYSTALECS-.327-12.5-12-C-TR
- added C11: 1u, LinnesLab-Passives:CAPACITOR0603
- C18: value 1u -> 4.7u
- renumbered C20 to C12
Connections:
- removed net A4/BATT: R16.1, R17.2
- removed net A6/TIA: J1.6
- removed net A7/PPG: J1.7
- removed net CD2: SD1.CARD_DETECT1
- removed net D29/LED.CTRL: J1.5
- removed net D5/CD1: SD1.CARD_DETECT
- removed net D7/SD.CS: SD1.CS
- removed net N$12: U3.OSCO, XTAL2.1
- removed net N$13: U3.OSCI, XTAL2.2
- removed net RXD: U1.P0.08
- removed net TXD: U1.P0.06
- new net A4/PPG: J1.7, U1.P0.28/AIN4
- new net A5/TIA: J1.5, U1.P0.29/AIN5
- new net A7/BATT: R16.1, R17.2, U1.P0.31/AIN7
- new net D30/LED.CTRL: J1.6, U1.P0.30/AIN6
- new net VIN1: C11.2, C18.2, CHRG1.VIN, LDO1.EN, LDO1.IN, R9.2
- net 3.3V: no longer C19.1, SD1.VDD, U3.VDD
- net D11/SW1: now also U1.P0.11
- net D15/SW2: now also U1.P0.15
- net D16/CS.OLED: now also U1.P0.16
- net D27/CHRG.STATUS: now also U1.P0.27
- net D3/RESET.OLED: now also U1.P0.03/AIN1
- net D4/DC.OLED: now also U1.P0.04/AIN2
- net GND: now also C11.1, C16.2; no longer C16.1, C19.2, C21.2, SD1.GND, SD1.GND1, SD1.VSS, U3.VSS
- net MISO: no longer SD1.DATA_OUT
- net MOSI: no longer SD1.DATA_IN
- net RXD.NRF: now also U1.P0.08
- net SCK: no longer SD1.SCLK
- net SCL: no longer U3.SCL
- net SDA: no longer U3.SDA
- net TXD.NRF: now also U1.P0.06
- net VIN: no longer C16.2, C18.2, CHRG1.VIN, LDO1.EN, LDO1.IN, R9.2
- net VLIPO: now also C16.1; no longer C21.1
Other:
- note added: "Diodes switch from LIPO power to USB when USB connected The USB charges battery then"
- note added: "R11 sets charge current I_charge = 1000V/R4 per MCP73831 document"
- note added: "Voltage divider used to measure battery voltage"
- note removed: "Back-up battery if desired"
- note removed: "Connect MISO, MOSI, and SCK to appropriate pins on microcontroller. Those are SPI pins and are generally prespecified. You have more flexibility with the SD.CS pin."
- note removed: "I2C Address = 0x68h"
- note removed: "Real-Time Clock"
- note removed: "SD card"
- moved on the sheet: C16, C18

Commit message: Finished Bottom and Top boards' first version
Parts:
- C11, C12: value 1u -> 47p
- C13: value 47p -> 100n
- C14: value 47p -> 4.7u
- C16: value 4.7u -> 1u
- C17: value 100n -> 1u
- renumbered SW4 to RESET, U4 to U3
Connections:
- net 3.3V: now also C15.2, C17.1; no longer C12.1, C17.2
- net DTR: now also C13.1; no longer C15.1
- net GND: now also C14.1, C15.1, C16.1, C17.2, C18.2; no longer C13.1, C14.2, C16.2, C17.1, C18.1
- net RESET: now also C13.2; no longer C15.2
- net USB+: now also C12.1; no longer C14.1
- net USB-: now also C11.2; no longer C13.2
- net VIN1: now also C14.2, C16.2; no longer C11.2, C18.2
- net VLIPO: now also C18.1; no longer C16.1
Other:
- moved on the sheet: C11, C12, C13, C14, C15, C16, C17, C18
