File: Hardware/Bottom/Tau-BOTTOM.sch (EAGLE design)
At the start: 31 parts, among them U1 AD5242-SO16

Commit message: Changes committed to top and bottom board
Parts:
- added J1: (no value), LinnesLab-Connectors:CONN_07
Connections:
- removed net LED.CTRL: U$4.A
- removed net TIA: C10.2, C15.1, OP4G$1.OUT, U1.W1
- new net A6/TIA: C10.2, C15.1, J1.5, OP4G$1.OUT, U1.W1
- new net A7/PPG: C21.2, J1.7, OP3G$1.OUT
- new net D29/LED.CTRL: J1.6, U$4.A
- net PPG: no longer C21.2, OP3G$1.OUT
Changed lines of the file:
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@@
 <part name="GND30" library="LinnesLab-Symbols" deviceset="GND" device=""/>
 <part name="SUPPLY24" library="LinnesLab-Symbols" deviceset="3.3V" device=""/>
+<part name="J1" library="LinnesLab-Connectors" deviceset="CONN_07" device=""/>
 </parts>
 <sheets>
@@
 <attribute name="VALUE" x="12.7" y="-32.766" size="1.778" layer="96" align="bottom-center"/>
 </instance>
+<instance part="J1" gate="G$1" x="99.06" y="-17.78" smashed="yes">
+<attribute name="VALUE" x="93.98" y="-27.686" size="1.778" layer="96" font="vector"/>
+<attribute name="NAME" x="93.98" y="-4.572" size="1.778" layer="95" font="vector"/>
+</instance>
 </instances>
 <busses>
@@
 </segment>
 </net>
-<net name="TIA" class="0">
+<net name="A6/TIA" class="0">
 <segment>
 <wire x1="124.46" y1="25.4" x2="119.38" y2="25.4" width="0.1524" layer="91"/>
@@
 <junction x="68.58" y="96.52"/>
 </segment>
+<segment>
+<pinref part="J1" gate="G$1" pin="5"/>
+<wire x1="104.14" y1="-12.7" x2="106.68" y2="-12.7" width="0.1524" layer="91"/>
+<label x="106.68" y="-12.7" size="1.27" layer="95" xref="yes"/>
+</segment>
 </net>
 <net name="PD.C" class="0">
@@
 </segment>
 </net>
-<net name="LED.CTRL" class="0">
+<net name="D29/LED.CTRL" class="0">
 <segment>
 <pinref part="U$4" gate="G$1" pin="A"/>
@@
 <wire x1="220.98" y1="27.94" x2="220.98" y2="35.56" width="0.1524" layer="91"/>
 <label x="220.98" y="35.56" size="1.27" layer="95" rot="R180" xref="yes"/>
+</segment>
+<segment>
+<pinref part="J1" gate="G$1" pin="6"/>
+<wire x1="104.14" y1="-10.16" x2="106.68" y2="-10.16" width="0.1524" layer="91"/>
+<label x="106.68" y="-10.16" size="1.27" layer="95" xref="yes"/>
 </segment>
 </net>
@@
 <label x="154.94" y="25.4" size="1.27" layer="95" xref="yes"/>
 <pinref part="U1" gate="G$1" pin="B2"/>
-</segment>
-<segment>
-<pinref part="C21" gate="G$1" pin="2"/>
-<wire x1="200.66" y1="99.06" x2="208.28" y2="99.06" width="0.1524" layer="91"/>
-<wire x1="208.28" y1="99.06" x2="208.28" y2="88.9" width="0.1524" layer="91"/>
-<pinref part="OP3" gate="G$1" pin="OUT"/>
-<wire x1="208.28" y1="88.9" x2="205.74" y2="88.9" width="0.1524" layer="91"/>
-<wire x1="208.28" y1="99.06" x2="208.28" y2="109.22" width="0.1524" layer="91"/>
-<junction x="208.28" y="99.06"/>
-<label x="208.28" y="109.22" size="1.27" layer="95" rot="R180" xref="yes"/>
-<label x="208.28" y="88.9" size="1.27" layer="95" xref="yes"/>
 </segment>
 </net>
@@
 </segment>
 </net>
+<net name="A7/PPG" class="0">
+<segment>
+<pinref part="C21" gate="G$1" pin="2"/>
+<wire x1="200.66" y1="99.06" x2="208.28" y2="99.06" width="0.1524" layer="91"/>
+<wire x1="208.28" y1="99.06" x2="208.28" y2="88.9" width="0.1524" layer="91"/>
+<pinref part="OP3" gate="G$1" pin="OUT"/>
+<wire x1="208.28" y1="88.9" x2="205.74" y2="88.9" width="0.1524" layer="91"/>
+<wire x1="208.28" y1="99.06" x2="208.28" y2="109.22" width="0.1524" layer="91"/>
+<junction x="208.28" y="99.06"/>
+<label x="208.28" y="109.22" size="1.27" layer="95" rot="R180" xref="yes"/>
+<label x="208.28" y="88.9" size="1.27" layer="95" xref="yes"/>
+</segment>
+<segment>
+<pinref part="J1" gate="G$1" pin="7"/>
+<wire x1="104.14" y1="-7.62" x2="106.68" y2="-7.62" width="0.1524" layer="91"/>
+<label x="106.68" y="-7.62" size="1.27" layer="95" xref="yes"/>
+</segment>
+</net>

Commit message: Bottom board nearly routed
Connections:
- removed net LED: Q1.C
- net LED.C: now also Q1.C
Changed lines of the file:
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@@
 <label x="22.86" y="96.52" size="1.27" layer="95" xref="yes"/>
+</segment>
+<segment>
+<wire x1="241.3" y1="27.94" x2="241.3" y2="30.48" width="0.1524" layer="91"/>
+<label x="241.3" y="30.48" size="1.27" layer="95" rot="R180" xref="yes"/>
+<pinref part="Q1" gate="G$1" pin="C"/>
 </segment>
 </net>
@@
 </segment>
 </net>
-<net name="LED" class="0">
-<segment>
-<wire x1="241.3" y1="27.94" x2="241.3" y2="30.48" width="0.1524" layer="91"/>
-<label x="241.3" y="30.48" size="1.27" layer="95" rot="R180" xref="yes"/>
-<pinref part="Q1" gate="G$1" pin="C"/>
-</segment>
-</net>

Commit message: Changes made to top and bottom board
Parts:
- removed J1: (no value), LinnesLab-Connectors:CONN_07
- added C1: 100n, LinnesLab-Passives:CAPACITOR0603
- added J2: (no value), LinnesLab-Connectors:CONN_07-1.27MM
Connections:
- removed net PPG: U1.B2
- net 3.3V: now also J2.4
- net A6/TIA: now also J2.6; no longer J1.5
- net A7/PPG: now also J2.7, U1.B2; no longer J1.7
- net D29/LED.CTRL: now also J2.5; no longer J1.6
- net GND: now also C1.1, J2.3
- net SCL: now also J2.2
- net SDA: now also J2.1
- net VREF: now also C1.2
Other:
- note added: "Castellated IMU breakout"
- note added: "Connection to digital potentiometer for dynamic control"
- note added: "Connection to optical sensor module"
- note added: "Connection to upper board"
- note added: "Vref Generator and Bypass Capacitors"

Commit message: Changes made to top and bottom board
Parts:
- added C2: 1u, LinnesLab-Passives:CAPACITOR0603
- added U3: PCF8523, LinnesLab-Clocks:PCF8523
- added XTAL2: 32.7680kHz, LinnesLab-Clocks:CRYSTALECS-.327-12.5-12-C-TR
Connections:
- new net N$12: U3.OSCO, XTAL2.1
- new net N$4: U3.OSCI, XTAL2.2
- net 3.3V: now also C2.1, U3.VDD
- net GND: now also C2.2, U3.VSS
- net SCL: now also U3.SCL
- net SDA: now also U3.SDA
Other:
- note added: "Back-up battery if desired"
- note added: "I2C Address = 0x68h"
- note added: "Real-Time Clock"

Commit message: Finished Bottom and Top boards' first version
Connections:
- net A6/TIA renamed A5/TIA
- net A7/PPG renamed A4/PPG
- net D29/LED.CTRL renamed D30/LED.CTRL
Changed lines of the file:
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@@
 </segment>
 </net>
-<net name="A6/TIA" class="0">
+<net name="A5/TIA" class="0">
 <segment>
 <wire x1="124.46" y1="25.4" x2="119.38" y2="25.4" width="0.1524" layer="91"/>
@@
 </segment>
 </net>
-<net name="D29/LED.CTRL" class="0">
+<net name="D30/LED.CTRL" class="0">
 <segment>
 <pinref part="U$4" gate="G$1" pin="A"/>
@@
 </segment>
 </net>
-<net name="A7/PPG" class="0">
+<net name="A4/PPG" class="0">
 <segment>
 <pinref part="C21" gate="G$1" pin="2"/>

Commit message: changes to bottom board
Other:
- note added: "Gain = -Rf (in pass band)"
- note added: "I_B = (3.3V - .6V)/(R_pot + R16) LED_current = I_B*Gain Current Gain of an NPN transistor is often written as HFE in datasheets"
Changed lines of the file:
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@@
 battery
 if desired</text>
+<text x="170.18" y="-10.16" size="1.778" layer="97">I_B = (3.3V - .6V)/(R_pot + R16)
+LED_current = I_B*Gain
+Current Gain of an NPN transistor is often written as HFE in datasheets</text>
+<text x="53.34" y="134.62" size="1.778" layer="97">Gain = -Rf (in pass band)</text>
 </plain>
 <instances>
